File: Hardware/KiCAD/TemperatureSensor/tempsensors.sch (KiCad schematic (older format))
At the start: 53 parts, among them J1 Conn_01x02, J2 Conn_01x02, J3 Conn_01x02, J4 Conn_01x02, U2 LD1117S33TR_SOT223, U3 MAX31856, U4 MAX31856, U5 MAX31856, U6 MAX31856

Commit message: working on temp sensors
Parts:
- added J5: Barrel_Jack, Connectors:BARREL_JACK, symbol Barrel_Jack
- C1, C10, C11, C12, C13, C14, C15, C16, C17, C18, C19, C2, C20, C21, C22, C3, C4, C5, C6, C7, C8, C9: footprint (none) -> Capacitors_SMD:C_0805
- D1, D10, D2, D5, D6, D9: footprint (none) -> Diodes_SMD:D_SOD-323
- D11: renamed from D?; footprint (none) -> Diodes_SMD:D_0805
- D3, D4, D7, D8: footprint (none) -> LEDs:LED_0603
- F1: renamed from F?; footprint (none) -> Fuse_Holders_and_Fuses:Fuseholder5x20_horiz_open_inline_Type-I
- J1, J2, J3, J4: footprint Terminal_Blocks:TerminalBlock_Pheonix_PT-3.5mm_2pol -> TemperatureSensor:Thermocouple_Pins
- R1, R10, R2, R3, R4, R5, R6, R7, R8, R9: footprint (none) -> Resistors_SMD:R_0603
- U2: footprint TO_SOT_Packages_SMD:SOT-223-3Lead_TabPin2 -> TO_SOT_Packages_THT:TO-220-3_Vertical
Connections:
- net GND: now also C1.2, C2.2, D11.2 (A), U2.1 (GND), J5.2, J5.3
- net VIN: now reaches C1.1, D11.1 (K), F1.1, U2.3 (VI)
- net +5V: no longer names the net of F1.2
- net +5V: now also J5.1
Other:
- moved on the sheet: C1, C2, D11, F1, U2
