File: Hardware/KiCAD/TemperatureSensor/TemperatureSensor.kicad_pcb (KiCad board)
At the start: 2 copper layers, 97.8 x 63.5 mm, 62 parts, among them J1 Conn_01x02, J2 Conn_01x02, J3 Conn_01x02, J4 Conn_01x02, J5 Barrel_Jack, J6 Conn_01x04, SW1 SW_Push, U1 ARDUINO_MICRO_SHIELD, U2 LD1117S33TR_SOT223, U3 MAX31856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

Commit message: test ltest layouayout
Parts:
- U1: footprint TemperatureSensor:ARDUINO_MICRO_SHIELD -> TemperatureSensor:ARDUINO_MICRO_SHIELD1
Connections:
- U1 pad 10: (no net) -> Net-(U1-Pad10)
- U1 pad 11: (no net) -> Net-(U1-Pad11)
- U1 pad 12: (no net) -> Net-(U1-Pad12)
- U1 pad 3.3V: (no net) -> Net-(U1-Pad3.3V)
- U1 pad 5V: (no net) -> Net-(U1-Pad5V)
- U1 pad A0: (no net) -> Net-(U1-PadA0)
- U1 pad A1: (no net) -> Net-(U1-PadA1)
- U1 pad A2: (no net) -> Net-(U1-PadA2)
- U1 pad A3: (no net) -> Net-(U1-PadA3)
- U1 pad A4: (no net) -> Net-(U1-PadA4)
- U1 pad A5: (no net) -> Net-(U1-PadA5)
- U1 pad AREF: (no net) -> Net-(U1-PadAREF)
- U1 pad MI: (no net) -> Net-(U1-PadMI)
- U1 pad MO: (no net) -> Net-(U1-PadMO)
- U1 pad RX: (no net) -> Net-(U1-PadRX)
- U1 pad SCK: (no net) -> Net-(U1-PadSCK)
- U1 pad SS: (no net) -> Net-(U1-PadSS)
- U1 pad TX: (no net) -> Net-(U1-PadTX)
- U3 pad 6: (no net) -> Net-(U3-Pad6)
- U3 pad 7: (no net) -> Net-(U3-Pad7)
- U4 pad 6: (no net) -> Net-(U4-Pad6)
- U4 pad 7: (no net) -> Net-(U4-Pad7)
- U5 pad 6: (no net) -> Net-(U5-Pad6)
- U5 pad 7: (no net) -> Net-(U5-Pad7)
- U6 pad 6: (no net) -> Net-(U6-Pad6)
- U6 pad 7: (no net) -> Net-(U6-Pad7)
Routing:
- net GND: track 0.00 -> 80.9 mm
- net VIN: track 43.1 -> 48.1 mm
- net Net-(F1-Pad2): track 13.9 -> 18.9 mm
- net Net-(U1-PadNC): track 0.00 -> 2.54 mm
- net SCK_3V3: track 84.6 -> 86.6 mm
- net Net-(SW1-Pad2): track 35.4 -> 34.7 mm
- net SDO: vias 5 -> 8
Other:
- rule trace_min: 0.2 -> 0.1
- rule via_min_size: 0.4 -> 0.2
